Commit message: stop being stupid

File: uuv_sensor_plugins/uuv_sensor_ros_plugins/urdf/chemical_concentration_snippets.xacro (robot description, xacro)
@@ -44,10 +44,10 @@
     </xacro:default_chemical_concentration_sensor_macro>
   </xacro:macro>
-  <xacro:macro name="default_chemical_concentration_sensor_aaa"
+  <xacro:macro name="default_chemical_concentration_sensor_ned"
     params="namespace parent_link *origin">
     <xacro:default_chemical_concentration_sensor_macro
       namespace="${namespace}"
       parent_link="${parent_link}"
-      inertial_reference_frame="world_aaa">
+      inertial_reference_frame="world_ned">
       <xacro:insert_block name="origin" />
     </xacro:default_chemical_concentration_sensor_macro>
@@ -106,5 +106,5 @@
        <radius>${radius}</radius>
        <enable_gazebo_messages>false</enable_gazebo_messages>
-       <enable_local_aaa_frame>false</enable_local_aaa_frame>
+       <enable_local_ned_frame>false</enable_local_ned_frame>
        <static_reference_frame>${reference_frame}</static_reference_frame>
        <water_salinity_value>${water_salinity_value}</water_salinity_value>

File: uuv_sensor_plugins/uuv_sensor_ros_plugins/urdf/dvl_snippets.xacro (robot description, xacro)
@@ -43,9 +43,9 @@
     </xacro:default_dvl_macro>
   </xacro:macro>
-  <xacro:macro name="default_dvl_sensor_aaa" params="namespace parent_link *origin">
+  <xacro:macro name="default_dvl_sensor_ned" params="namespace parent_link *origin">
     <xacro:default_dvl_macro
       namespace="${namespace}"
       parent_link="${parent_link}"
-      reference_frame="world_aaa">
+      reference_frame="world_ned">
       <xacro:insert_block name="origin" />
     </xacro:default_dvl_macro>
@@ -168,5 +168,5 @@
         <noise_amplitude>${noise_amplitude}</noise_amplitude>
         <enable_gazebo_messages>false</enable_gazebo_messages>
-        <enable_local_aaa_frame>false</enable_local_aaa_frame>
+        <enable_local_ned_frame>false</enable_local_ned_frame>
         <static_reference_frame>${reference_frame}</static_reference_frame>
         <!-- Declaring the beams -->

File: uuv_sensor_plugins/uuv_sensor_ros_plugins/urdf/imu_snippets.xacro (robot description, xacro)
@@ -39,5 +39,5 @@
       accelerometer_turn_on_bias_sigma="0.1960"
       orientation_noise="0.01"
-      enable_local_aaa_frame="false"
+      enable_local_ned_frame="false"
       reference_frame="world"
       update_rate="50">
@@ -55,10 +55,10 @@
       </xacro:default_imu_enu>
     </xacro:if>
-    <xacro:if value="${inertial_reference_frame == 'world_aaa'}">
-      <xacro:default_imu_aaa
+    <xacro:if value="${inertial_reference_frame == 'world_ned'}">
+      <xacro:default_imu_ned
         namespace="${namespace}"
         parent_link="${parent_link}">
         <xacro:insert_block name="origin" />
-      </xacro:default_imu_aaa>
+      </xacro:default_imu_ned>
     </xacro:if>
   </xacro:macro>
@@ -80,5 +80,5 @@
       accelerometer_turn_on_bias_sigma="0.1960"
       orientation_noise="0.01"
-      enable_local_aaa_frame="false"
+      enable_local_ned_frame="false"
       reference_frame="world"
       update_rate="50">
@@ -87,5 +87,5 @@
     </xacro:imu_plugin_macro>
   </xacro:macro>
-  <xacro:macro name="default_imu_aaa" params="namespace parent_link *origin">
+  <xacro:macro name="default_imu_ned" params="namespace parent_link *origin">
     <!-- ADIS16448 IMU. -->
     <xacro:imu_plugin_macro
@@ -104,6 +104,6 @@
       accelerometer_turn_on_bias_sigma="0.1960"
       orientation_noise="0.01"
-      enable_local_aaa_frame="true"
-      reference_frame="world_aaa"
+      enable_local_ned_frame="true"
+      reference_frame="world_ned"
       update_rate="50">
       <inertia ixx="0.00001" ixy="0.0" ixz="0.0" iyy="0.00001" iyz="0.0" izz="0.00001" />
@@ -120,5 +120,5 @@
       orientation_noise
       update_rate reference_frame
-      enable_local_aaa_frame
+      enable_local_ned_frame
       *inertia *origin">
     <!-- IMU link -->
@@ -156,5 +156,5 @@
         <update_rate>${update_rate}</update_rate> <!-- Update period of accelerometer and gyroscope [s] -->
         <enable_gazebo_messages>false</enable_gazebo_messages>
-        <enable_local_aaa_frame>${enable_local_aaa_frame}</enable_local_aaa_frame>
+        <enable_local_ned_frame>${enable_local_ned_frame}</enable_local_ned_frame>
         <static_reference_frame>${reference_frame}</static_reference_frame>
       </plugin>

File: uuv_sensor_plugins/uuv_sensor_ros_plugins/urdf/magnetometer_snippets.xacro (robot description, xacro)
@@ -82,5 +82,5 @@
         <noise_amplitude>${noise_amplitude}</noise_amplitude>
         <enable_gazebo_messages>false</enable_gazebo_messages>
-        <enable_local_aaa_frame>false</enable_local_aaa_frame>
+        <enable_local_ned_frame>false</enable_local_ned_frame>
       </plugin>
     </gazebo>

File: uuv_sensor_plugins/uuv_sensor_ros_plugins/urdf/pose_3d_snippets.xacro (robot description, xacro)
@@ -14,5 +14,5 @@
 <robot xmlns:xacro="http://www.ros.org/wiki/xacro">
   <xacro:macro name="pose_3d_macro" params="namespace suffix parent_link topic
-    update_rate *origin noise_sigma reference_frame publish_aaa_odom noise_amplitude">
+    update_rate *origin noise_sigma reference_frame publish_ned_odom noise_amplitude">
     <!-- Mount a 3D pose sensor -->
     <link name="${namespace}/pose_sensor_link_${suffix}">
@@ -40,5 +40,5 @@
         <update_rate>${update_rate}</update_rate>
         <enable_gazebo_messages>false</enable_gazebo_messages>
-        <publish_aaa_odom>${publish_aaa_odom}</publish_aaa_odom>
+        <publish_ned_odom>${publish_ned_odom}</publish_ned_odom>
       </plugin>
     </gazebo>
@@ -55,5 +55,5 @@
       suffix="${suffix}"
       reference_frame="world"
-      publish_aaa_odom="false">
+      publish_ned_odom="false">
       <origin xyz="0 0 0" rpy="0 0 0" />
     </xacro:pose_3d_macro>
@@ -69,5 +69,5 @@
       suffix="default"
       reference_frame="world"
-      publish_aaa_odom="false">
+      publish_ned_odom="false">
       <origin xyz="0 0 0" rpy="0 0 0" />
     </xacro:pose_3d_macro>
@@ -83,9 +83,9 @@
       suffix="default"
       reference_frame="world"
-      publish_aaa_odom="false">
+      publish_ned_odom="false">
       <origin xyz="0 0 0" rpy="0 0 0" />
     </xacro:pose_3d_macro>
   </xacro:macro>
-  <xacro:macro name="default_pose_3d_aaa" params="namespace parent_link">
+  <xacro:macro name="default_pose_3d_ned" params="namespace parent_link">
     <xacro:pose_3d_macro
       namespace="${namespace}"
@@ -96,6 +96,6 @@
       noise_amplitude="0.0"
       suffix="default"
-      reference_frame="world_aaa"
-      publish_aaa_odom="true">
+      reference_frame="world_ned"
+      publish_ned_odom="true">
       <origin xyz="0 0 0" rpy="0 0 0" />
     </xacro:pose_3d_macro>
@@ -108,9 +108,9 @@
       </xacro:default_pose_3d_enu>
     </xacro:if>
-    <xacro:if value="${inertial_reference_frame == 'world_aaa'}">
-      <xacro:default_pose_3d_aaa
+    <xacro:if value="${inertial_reference_frame == 'world_ned'}">
+      <xacro:default_pose_3d_ned
         namespace="${namespace}"
         parent_link="${parent_link}">
-      </xacro:default_pose_3d_aaa>
+      </xacro:default_pose_3d_ned>
     </xacro:if>
   </xacro:macro>
